Commit message: Modified learning notes
Signed-off-by: daveohs <wellclosedoor@gmail.com>

File: urdf/manipulator.xacro (robot description, xacro)
@@ -15,7 +15,7 @@
   ===================================================================
   -->
-  <material name="white"><color rgba="1 1 1 1"/></material>
-  <material name="blue"><color rgba="0.2 0.2 1 1"/></material>
-  <material name="grey"><color rgba="0.5 0.5 0.5 1"/></material>
+  <material name="White"><color rgba="1 1 1 1"/></material>
+  <material name="Blue"><color rgba="0.2 0.2 1 1"/></material>
+  <material name="Grey"><color rgba="0.5 0.5 0.5 1"/></material>
   <!--
   ===================================================================
