Commit message: Added package for moveit
Signed-off-by: daveohs <wellclosedoor@gmail.com>

File: my_manipulator/urdf/manipulator.xacro (robot description, xacro)
@@ -29,5 +29,5 @@
       <visual>
         <geometry>
-          <mesh filename="package://manipulator/meshes/${link_name}.stl" scale="${mesh_scale}"/>
+          <mesh filename="package://my_manipulator/meshes/${link_name}.stl" scale="${mesh_scale}"/>
         </geometry>
         <material name="${gazebo_material}"/>
@@ -35,5 +35,5 @@
       <collision>
         <geometry>
-          <mesh filename="package://manipulator/meshes/${link_name}.stl" scale="${mesh_scale}"/>
+          <mesh filename="package://my_manipulator/meshes/${link_name}.stl" scale="${mesh_scale}"/>
         </geometry>
       </collision>

File: my_manipulator/urdf/manipulator_real.urdf.xacro (robot description, xacro)
@@ -6,5 +6,5 @@
   <xacro:arg name="dry_run" default="false"/>
   <!-- 1. 공통 로봇 모델 포함 -->
-  <xacro:include filename="$(find manipulator)/urdf/manipulator.xacro" />
+  <xacro:include filename="$(find my_manipulator)/urdf/manipulator.xacro" />
   <!--
   ===================================================================

File: my_manipulator/urdf/manipulator_sim.urdf.xacro (robot description, xacro)
@@ -2,5 +2,5 @@
 <robot xmlns:xacro="http://www.ros.org/wiki/xacro" name="manipulator">
   <!-- 1. 공통 로봇 모델 포함 -->
-  <xacro:include filename="$(find manipulator)/urdf/manipulator.xacro" />
+  <xacro:include filename="$(find my_manipulator)/urdf/manipulator.xacro" />
   <!--
   ===================================================================
@@ -31,5 +31,5 @@
   <gazebo>
     <plugin name="gazebo_ros2_control" filename="libgazebo_ros2_control.so">
-      <parameters>$(find manipulator)/config/my_controllers.yaml</parameters>
+      <parameters>$(find my_manipulator)/config/my_controllers.yaml</parameters>
     </plugin>
   </gazebo>
